File: Raspi_HAT/Raspi_HAT.kicad_pcb (KiCad board)
At the start: 2 copper layers, 65 x 56 mm, 36 parts, among them J1 GPIO, J10 PIRANI_JST, J11 RPM_JST, J2 ADC1_Conn_01x10_Pin, J3 DAC1_Conn_01x06_Pin, J5 VALVE, J6 TURBO_EN, J8 UART_JST, J9 MFC_JST, K1 G5V-1 5V, Q1 BC847B, Q2 BC847B, U1 CAT24C256, U2 EL817 (SMD), U3 LM358

Commit message: Add web dashboard (SSE + stdlib server), mac launchers, app icons
Other:
- board size 65 x 56 mm -> 65 x 76 mm
Changed lines of the file:
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@@
 	(gr_line
 		(start 100 81)
-		(end 100 97)
+		(end 100 117)
 		(stroke
 			(width 0.1)
@@
 	)
 	(gr_arc
-		(start 103 100)
-		(mid 100.87868 99.12132)
-		(end 100 97)
+		(start 103 120)
+		(mid 100.87868 119.12132)
+		(end 100 117)
 		(stroke
 			(width 0.1)
@@
 	)
 	(gr_line
-		(start 103 100)
-		(end 162 100)
+		(start 103 120)
+		(end 162.127399 120)
 		(stroke
 			(width 0.1)
@@
 	)
 	(gr_arc
-		(start 165 97)
-		(mid 164.12132 99.12132)
-		(end 162 100)
+		(start 165 117.127399)
+		(mid 164.158634 119.158634)
+		(end 162.127399 120)
 		(stroke
 			(width 0.1)
@@
 	)
 	(gr_line
-		(start 165 97)
+		(start 165 117.127399)
 		(end 165 47)
 		(stroke
